File: Hardware/Example_Implementation/Module_Carrier_Board/STM32L4xx-v1.2.0.brd (EAGLE design)
At the start: 78.7 x 50.8 mm, 66 parts, among them CON2 TC2030-CTX-NL, IC4 ATECC608A, Q1 CSTCE8M00G55-R0, Q3 32.768kHz, U1 STM32L475VGT6, U2 MX25R3235FM1IH0

Commit message: Adding v1.2.0 (& remove v1.1.0) files for MCB & MEB
Parts:
- TP1, TP2: value TEST-POINT-50R-PTH -> TEST_POINT-50R-PTH; device mbed-HDK:TP50-PTH -> mbed-HDK-Test:TP50-PTH
- TP10, TP11, TP12, TP13, TP14, TP15, TP16, TP17, TP18, TP19, TP20, TP21, TP22, TP23, TP24, TP25, TP26, TP27, TP28, TP29, TP3, TP30, TP31, TP32, TP33, TP34, TP35, TP36, TP37, TP38, TP39, TP4, TP40, TP41, TP42, TP43, TP44, TP45, TP5, TP6, TP7, TP8, TP9: device testpad:TP06R -> mbed-HDK-Test:TP06R
- U1: device STM32L475VGT6:QFP50P1600X1600X160-100N -> SnapEDA:QFP50P1600X1600X160-100N
Connections:
- net PA0: now also MOD1.19; no longer MOD1.18
- net PA1: now also MOD1.20; no longer MOD1.19
- net PB0: now also MOD1.18; no longer MOD1.20
Routing:
- net PB0: track 48.1 -> 46.6 mm
- net PB6: track 61.0 -> 62.5 mm
- net PB7: track 62.7 -> 64.1 mm
- net PB5: track 49.4 -> 50.5 mm
- net +3.3V: track 239.7 -> 238.6 mm
- net PA0: track 46.5 -> 45.8 mm
Other:
- board text added: "GND 3V3 TGT_SWDIO TGT_SWCLK TGT_NRESET TGT_TX TGT_RX PA2 PA3 PB7 PB6 PB5 PA6 PA5 PB0 PA0 PA1"
- board text added: "Module Carrier Board STM32L v1.2.0"
- board text removed: "GND 3V3 TGT_SWDIO TGT_SWCLK TGT_NRESET TGT_TX TGT_RX PA2 PA3 PB7 PB6 PB5 PA6 PA5 PA0 PA1 PB0"
- board text removed: "Module Carrier Board STM32L v1.1.0"
