File: Hardware/Example_Implementation/Module_Carrier_Board/STM32L4xx-v1.2.0.sch (EAGLE design)
At the start: 66 parts, among them CON2 TC2030-CTX-NL, IC4 ATECC608A, Q1 CSTCE8M00G55-R0, Q3 32.768kHz, U1 STM32L475VGT6, U2 MX25R3235FM1IH0

Commit message: Adding v1.2.0 (& remove v1.1.0) files for MCB & MEB
Parts:
- TP1, TP2: value TEST-POINT-50R-PTH -> TEST_POINT-50R-PTH; device mbed-HDK:TEST-POINT-50R-PTH -> mbed-HDK-Test:TEST_POINT-50R-PTH
- TP10, TP11, TP12, TP13, TP14, TP15, TP16, TP17, TP18, TP19, TP20, TP21, TP22, TP23, TP24, TP25, TP26, TP27, TP28, TP29, TP3, TP30, TP31, TP32, TP33, TP34, TP35, TP36, TP37, TP38, TP39, TP4, TP40, TP41, TP42, TP43, TP44, TP45, TP5, TP6, TP7, TP8, TP9: device testpad:PTR1TP06R -> mbed-HDK-Test:PTR1TP06R
- U1: device STM32L475VGT6:STM32L475VGT6 -> SnapEDA:STM32L475VGT6
Connections:
- net PA0: now also MOD1.AIN1/GROVE; no longer MOD1.AIN0/POT
- net PA1: now also MOD1.AIN2/GROVE; no longer MOD1.AIN1/GROVE
- net PA3: now also U1ETH.UART2-RX/AIN8/PA3; no longer U1ETH.UART2-TX/AIN8/PA3
- net PB0: now also MOD1.AIN0/POT; no longer MOD1.AIN2/GROVE
