File: Hardware/Example_Implementation/Module_Expansion_Board/MEB-Quectel-BG96-v1.2.0.brd (EAGLE design)
At the start: 83.8 x 78.7 mm, 87 parts, among them CON1 SMA-142-0701-801/806, CON2 47346-0001, CON3 FC68148S, CON4 SMA-142-0701-801/806, IC1 MIC29302WU, IC2 74AHC1G08DCK, J1 SF56S006V4BR2000, T1 BC850C,215, T2 BC850C,215, T3 BC850C,215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

Commit message: Adding v1.2.0 (& remove v1.1.0) files for MCB & MEB
Parts:
- removed TP16, TP19: TEST_POINT-50R-SMD, mbed-HDK-Test:TP50-SMD
- C13, C14: device rcl:150CLZ-0810 -> mbed-HDK-RLC:PANASONIC_F
- IC2: value 74AHC1G08DCK -> 74LVC1G08DCK; device 74xx-little-us:SC70-5 -> mbed-HDK-IC:SC70-5
- moved C14 0.63 mm to (52.1, 57.3)
Connections:
- removed net N$10: MOD1.37, TP16.TP
- removed net N$38 (its old number): BRD1.18, BRD1.58
- removed net N$39: BRD1.19, BRD1.59
- removed net N$48: MOD1.36, TP19.TP
- new net MCU_CTS_1V8: MOD1.37, U1.6
- new net MCU_CTS_3V3: BRD1.18, U1.15
- new net MCU_RTS_1V8: MOD1.36, U1.7
- new net MCU_RTS_3V3: BRD1.19, U1.14
- net +1.8V: now also R23.2
- net SIM_VDD: no longer R23.2
Routing:
- net MCU_CTS_3V3: track 0.00 -> 61.4 mm, vias 0 -> 2
- net MCU_RTS_3V3: track 0.00 -> 60.9 mm, vias 0 -> 2
- net MCU_CTS_1V8: track 0.00 -> 55.8 mm, vias 0 -> 2
- net MCU_RTS_1V8: track 0.00 -> 54.2 mm, vias 0 -> 2
- net +1.8V: track 57.5 -> 98.8 mm, vias 4 -> 7
- net N$10: track 7.22 -> 0.00 mm
- net N$48: track 5.31 -> 0.00 mm
- net N$41: track 51.4 -> 46.7 mm
- net N$39: track 2.54 -> 0.00 mm
- net N$38 (its old number): track 2.54 -> 0.00 mm
- net MCU_TX_3V3: track 28.9 -> 30.7 mm
- net MCU_RX_3V3: track 29.1 -> 30.3 mm
- net N$71: track 15.1 -> 16.1 mm
- net DBG_RXD_1V8: track 56.4 -> 55.7 mm
- net SIM_VDD: track 66.8 -> 66.1 mm
Other:
- board text added: "Quectel BG96 v1.2.0"
- board text removed: "Quectel BG96 v1.1.0"
